File: hardware/co2-sensor.sch (EAGLE design)
At the start: 21 parts, among them IC1 LM1117IMPX-3.3, J1 MH-Z19, U1 esp12e, U2 dht22, U3 BMP280

Commit message: .
Parts:
- removed R4: 10k, rcl:R-EU_M0805
- removed U2: dht22, RHT03_DHT-22_AM2302:RHT03_DHT-22_AM2302WIRED
Connections:
- net +5V: no longer R4.2, U2.VDD
- net DHT22: no longer R4.1, U2.DATA
- net GND: no longer U2.GND
Changed lines of the file:
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@@
 <part name="+3V3" library="supply1" library_urn="urn:adsk.eagle:library:371" deviceset="+3V3" device=""/>
 <part name="C2" library="rcl" library_urn="urn:adsk.eagle:library:334" deviceset="CPOL-EU" device="CT3216" package3d_urn="urn:adsk.eagle:package:23327/2" value="100mF"/>
-<part name="U2" library="RHT03_DHT-22_AM2302" deviceset="RHT03_DHT-22_AM2302" device="WIRED" value="dht22"/>
-<part name="P+4" library="supply1" library_urn="urn:adsk.eagle:library:371" deviceset="+5V" device=""/>
-<part name="GND10" library="supply1" library_urn="urn:adsk.eagle:library:371" deviceset="GND" device=""/>
 <part name="C3" library="rcl" library_urn="urn:adsk.eagle:library:334" deviceset="C-EU" device="C0805" package3d_urn="urn:adsk.eagle:package:23617/2" value="100n"/>
 <part name="GND8" library="supply1" library_urn="urn:adsk.eagle:library:371" deviceset="GND" device=""/>
@@
 <part name="C4" library="rcl" library_urn="urn:adsk.eagle:library:334" deviceset="C-EU" device="C0805" package3d_urn="urn:adsk.eagle:package:23617/2" value="10u"/>
 <part name="R3" library="rcl" library_urn="urn:adsk.eagle:library:334" deviceset="R-EU_" device="M0805" package3d_urn="urn:adsk.eagle:package:23556/1" value="4.7k"/>
-<part name="R4" library="rcl" library_urn="urn:adsk.eagle:library:334" deviceset="R-EU_" device="M0805" package3d_urn="urn:adsk.eagle:package:23556/1" value="10k"/>
 <part name="U$1" library="USB-C" deviceset="USB-C" device=""/>
 <part name="GND1" library="supply1" library_urn="urn:adsk.eagle:library:371" deviceset="GND" device=""/>
@@
 <attribute name="VALUE" x="54.483" y="-14.7574" size="1.778" layer="96"/>
 </instance>
-<instance part="U2" gate="G$1" x="17.78" y="-73.66" smashed="yes" rot="MR0">
-<attribute name="NAME" x="22.86" y="-62.23" size="1.27" layer="94" rot="MR0"/>
-<attribute name="VALUE" x="22.86" y="-86.36" size="1.27" layer="94" rot="MR0"/>
-</instance>
-<instance part="P+4" gate="1" x="45.72" y="-60.96" smashed="yes" rot="MR90">
-<attribute name="VALUE" x="40.64" y="-63.5" size="1.778" layer="96" rot="MR180"/>
-</instance>
-<instance part="GND10" gate="1" x="33.02" y="-83.82" smashed="yes" rot="MR0">
-<attribute name="VALUE" x="35.56" y="-86.36" size="1.778" layer="96" rot="MR0"/>
-</instance>
 <instance part="C3" gate="G$1" x="60.96" y="-10.16" smashed="yes">
 <attribute name="NAME" x="62.484" y="-9.779" size="1.778" layer="95"/>
@@
 <attribute name="NAME" x="146.2786" y="-24.13" size="1.778" layer="95" rot="R270"/>
 <attribute name="VALUE" x="141.478" y="-24.13" size="1.778" layer="96" rot="R270"/>
-</instance>
-<instance part="R4" gate="G$1" x="35.56" y="-66.04" smashed="yes" rot="MR90">
-<attribute name="NAME" x="37.0586" y="-69.85" size="1.778" layer="95" rot="MR90"/>
-<attribute name="VALUE" x="32.258" y="-69.85" size="1.778" layer="96" rot="MR90"/>
 </instance>
 <instance part="U$1" gate="G$1" x="15.24" y="-2.54" smashed="yes">
@@
 <pinref part="C2" gate="G$1" pin="-"/>
 <wire x1="53.34" y1="-17.78" x2="53.34" y2="-15.24" width="0.1524" layer="91"/>
-</segment>
-<segment>
-<pinref part="U2" gate="G$1" pin="GND"/>
-<pinref part="GND10" gate="1" pin="GND"/>
-<wire x1="33.02" y1="-81.28" x2="27.94" y2="-81.28" width="0.1524" layer="91"/>
 </segment>
 <segment>
@@
 </segment>
 <segment>
-<pinref part="R4" gate="G$1" pin="2"/>
-<pinref part="P+4" gate="1" pin="+5V"/>
-<wire x1="43.18" y1="-60.96" x2="35.56" y2="-60.96" width="0.1524" layer="91"/>
-<pinref part="U2" gate="G$1" pin="VDD"/>
-<wire x1="35.56" y1="-60.96" x2="27.94" y2="-60.96" width="0.1524" layer="91"/>
-<wire x1="27.94" y1="-60.96" x2="27.94" y2="-66.04" width="0.1524" layer="91"/>
-<junction x="35.56" y="-60.96"/>
-</segment>
-<segment>
 <pinref part="LED1" gate="G$1" pin="VDD"/>
 <pinref part="P+2" gate="1" pin="+5V"/>
@@
 <net name="DHT22" class="0">
 <segment>
-<pinref part="U2" gate="G$1" pin="DATA"/>
-<wire x1="27.94" y1="-71.12" x2="35.56" y2="-71.12" width="0.1524" layer="91"/>
-<label x="40.64" y="-71.12" size="1.016" layer="95" rot="MR180" xref="yes"/>
-<pinref part="R4" gate="G$1" pin="1"/>
-<wire x1="35.56" y1="-71.12" x2="40.64" y2="-71.12" width="0.1524" layer="91"/>
-<junction x="35.56" y="-71.12"/>
-</segment>
-<segment>
 <pinref part="U1" gate="G$1" pin="GPIO12"/>
